File: PCB/Controllers/Controllers.kicad_pcb (KiCad board)
At the start: 2 copper layers, 120.7 x 57.1 mm, 9 parts, among them J1 Main_Connector, SW1 A, SW2 BL, SW3 B, SW4 BR, U1 COM-09032

Commit message: generated gerbers and ordered PCB (#9)
Routing:
- net +3V3: track 228.5 -> 229.8 mm
Other:
- outline, holes or cut-outs redrawn
